Commit message: add rover description package

File: rover_description/urdf/rover.urdf (robot description, URDF)
Before this commit: robot rover, 9 links, 8 joints
Joints:
- joint left_hub_joint: axis 0 1 0 -> 0 -1 0
- joint right_back_joint: axis 0 1 0 -> 0 -1 0
- joint right_front_joint: axis 0 1 0 -> 0 -1 0
- joint right_hub_joint: axis 0 1 0 -> 0 -1 0; origin xyz=0.24617 -0.26216 -0.02379 rpy=0 0 0 -> xyz=0.24617 -0.25899 -0.02379 rpy=0 0 0
- joint right_mid_joint: axis 0 1 0 -> 0 -1 0
